Commit message: Final version of pixel iteration and folder resctructure

File: my_robot/urdf/my_robot.xacro (robot description, xacro)
@@ -1,10 +1,23 @@
 <?xml version='1.0'?>
+<!--Drive robot straight, might be swaying one direction a little bit more-->
 <robot name="my_robot" xmlns:xacro="http://www.ros.org/wiki/xacro">
   <xacro:include filename="$(find my_robot)/urdf/my_robot.gazebo"/>
+  <gazebo reference="chassis">
+    <material>Gazebo/Green</material>
+  </gazebo>
+  <gazebo reference="left_wheel">
+    <material>Gazebo/FlatBlack</material>
+  </gazebo>
+  <gazebo reference="right_wheel">
+    <material>Gazebo/FlatBlack</material>
+  </gazebo>
+  <gazebo reference="camera">
+    <material>Gazebo/Indigo</material>
+  </gazebo>
   <link name="robot_footprint"></link>
   <joint name="robot_footprint_joint" type="fixed">
-  <origin xyz="0 0 0" rpy="0 0 0" />
-  <parent link="robot_footprint"/>
-  <child link="chassis" />
+    <origin xyz="0 0 0" rpy="0 0 0" />
+    <parent link="robot_footprint"/>
+    <child link="chassis" />
   </joint>
   <link name='chassis'>
@@ -12,5 +25,5 @@
       <inertial>
         <mass value="15.0"/>
-        <origin xyz="0.0 0 0" rpy=" 0 0 0"/>
+        <origin xyz="0.0 0 0.05" rpy=" 0 0 0"/>
         <inertia
                 ixx="0.1" ixy="0" ixz="0"
@@ -20,38 +33,47 @@
       </inertial>
       <collision name='collision'>
-        <origin xyz="0 0 0" rpy=" 0 0 0"/>
-        <geometry>
-              <box size=".4 .2 .1"/>
+        <origin xyz="0 0 0.05" rpy="0 0 0"/>
+        <geometry>
+              <cylinder radius="0.35" length="0.15"/>
         </geometry>
       </collision>
       <visual name='chassis_visual'>
-        <origin xyz="0 0 0" rpy=" 0 0 0"/>
-        <geometry>
-              <box size=".4 .2 .1"/>
-        </geometry>
+        <origin xyz="0 0 0.05" rpy="0 0 0"/>
+        <geometry>
+              <cylinder radius="0.35" length="0.15"/>
+        </geometry>
+        <material name="green">
+          <color rgba="0.1 0.8 0.2 1"/>
+        </material>
       </visual>
-      <collision name='back_caster_collision'>
-        <origin xyz="-0.15 0 -0.05" rpy=" 0 0 0"/>
-        <geometry>
-              <sphere radius="0.0499"/>
+      <collision name="front_caster_collision">
+        <origin xyz="0.25 0 0" rpy="0 0 0"/>
+        <geometry>
+            <sphere radius="0.075"/>
         </geometry>
       </collision>
-      <visual name='back_caster_visual'>
-        <origin xyz="-0.15 0 -0.05" rpy=" 0 0 0"/>
-        <geometry>
-              <sphere radius="0.05"/>
-        </geometry>
+      <visual name="front_caster_visual">
+        <origin xyz="0.25 0 0" rpy="0 0 0"/>
+        <geometry>
+            <sphere radius="0.075"/>
+        </geometry>
+        <material name="grey">
+          <color rgba="0.5 0.6 0.7 1"/>
+        </material>
       </visual>
-      <collision name='front_caster_collision'>
-        <origin xyz="0.15 0 -0.05" rpy=" 0 0 0"/>
-        <geometry>
-              <sphere radius="0.0499"/>
+      <collision name="back_caster_collision">
+        <origin xyz="-0.25 0 0" rpy="0 0 0"/>
+        <geometry>
+            <sphere radius="0.075"/>
         </geometry>
       </collision>
-      <visual name='front_caster_visual'>
-        <origin xyz="0.15 0 -0.05" rpy=" 0 0 0"/>
-        <geometry>
-              <sphere radius="0.05"/>
-        </geometry>
+      <visual name="back_caster_visual">
+        <origin xyz="-0.25 0 0" rpy="0 0 0"/>
+        <geometry>
+            <sphere radius="0.075"/>
+        </geometry>
+        <material name="grey">
+          <color rgba="0.5 0.6 0.7 1"/>
+        </material>
       </visual>
   </link>
@@ -70,16 +92,17 @@
       <origin xyz="0 0 0" rpy="0 1.5707 1.5707"/>
         <geometry>
-          <cylinder radius="0.1" length="0.05"/>
-        </geometry>
+          <cylinder radius="0.075" length="0.05"/>
+        </geometry>
+      <material name="black"/>
     </visual>
     <collision name="left_wheel_collision">
       <origin xyz="0 0 0" rpy="0 1.5707 1.5707"/>
         <geometry>
-          <cylinder radius="0.1" length="0.05"/>
+          <cylinder radius="0.075" length="0.05"/>
         </geometry>
     </collision>
 	</link>
   <joint type="continuous" name="left_wheel_hinge">
-    <origin xyz="0 0.15 0" rpy="0 0 0"/>
+    <origin xyz="-0.05 0.3 0" rpy="0 0 0"/>
     <child link="left_wheel"/>
     <parent link="chassis"/>
@@ -102,16 +125,19 @@
         <origin xyz="0 0 0" rpy="0 1.5707 1.5707"/>
         <geometry>
-            <cylinder radius="0.1" length="0.05"/>
-        </geometry>
+            <cylinder radius="0.075" length="0.05"/>
+        </geometry>
+        <material name="black">
+          <color rgba="0 0 0 1"/>
+        </material>
     </visual>
     <collision name="right_wheel_collision">
         <origin xyz="0 0 0" rpy="0 1.5707 1.5707"/>
         <geometry>
-            <cylinder radius="0.1" length="0.05"/>
+            <cylinder radius="0.075" length="0.05"/>
         </geometry>
     </collision>
   </link>
   <joint type="continuous" name="right_wheel_hinge">
-    <origin xyz="0 -0.15 0" rpy="0 0 0"/>
+    <origin xyz="-0.05 -0.3 0" rpy="0 0 0"/>
     <child link="right_wheel"/>
     <parent link="chassis"/>
@@ -136,4 +162,7 @@
         <box size="0.05 0.05 0.05"/>
       </geometry>
+      <material name="purple">
+        <color rgba="0.4 0.3 0.8 0.79"/>
+      </material>
     </visual>
     <collision name="camera_collision">
@@ -145,5 +174,5 @@
   </link>
   <joint type="fixed" name="camera_joint">
-    <origin xyz="0.2 0 0" rpy="0 0 0"/>
+    <origin xyz="0.35 0 0.025" rpy="0 0 0"/>
     <child link="camera"/>
     <parent link="chassis"/>
@@ -175,5 +204,5 @@
   </link>
   <joint type="fixed" name="hokuyo_joint">
-    <origin xyz="0.15 0 0.1" rpy="0 0 0"/>
+    <origin xyz="0.0 0 0.15" rpy="0 0 0"/>
     <child link="hokuyo"/>
     <parent link="chassis"/>
